File: bloxa.sch (EAGLE design)
At the start: 93 parts, among them CON1 CON-4P-JST_GH-RA, CON2 CON-4P-JST_GH-RA, IC1 MCP9700-SC70-5, IC2 TPD3S014DBVR-SOT23-6, IC3 TJA1051(X)/3-SO8, J1 CONNECTION, J2 CONNECTION, Q1 BUK9K6R2-40E,115, Q2 BUK9K6R2-40E,115, Q3 BUK9K6R2-40E,115

Commit message: attribute updated
Parts:
- D1: value PTVS36VP1UP,115-36V-SOD128 -> PTVS33VP1UTP,115-36V-SOD128; device TVS_diodes:PTVS36VP1UP,115-36V-SOD128 -> TVS_diodes:PTVS33VP1UTP,115-36V-SOD128
- LED1: device myxa_masterlib:LED-GREEN-0402 -> rc:LED-0402
- LED2: device myxa_masterlib:LED-GREEN-0402 -> rc:LED-0402; COLOR (none) -> GREEN; DIGIKEY# (none) -> 1830-IN-S42BT5GCT-ND; MANF (none) -> Inolux; MANF# (none) -> IN-S42BT5G
- LED3, LED4: device myxa_masterlib:LTST-C19HE1WT -> misc:LTST-C19HE1WT
Other:
- note added: "-Current shunts replaced (5 mOhms replaced with 10 mOhms)- -Overcurrent protection added. Itrip is ~35 A -RCPWM th connector replaced with smd solder pads -Some design notes added to the schematic -TVS diode (D1) replaced with one that has lower breaksdown voltage"
- note added: "The table is valid for 26.4 V supply voltage which is the same as a discharched 8S Li-ion battery"
- note removed: "-Current shunts replaced (5 mOhms replaced with 10 mOhms)- -Overcurrent protection added. Itrip is ~35 A -RCPWM th connector replaced with smd solder pads -Some design notes added to the schematic"
- note removed: "The table is valid for 26.4 V supply voltage which is discharched 8S battery"
- moved on the sheet: C10, D1, LED3, LED4, PAD42, PAD43, R3, R5, R6, R7

Commit message: resolving conflicts
Parts:
- removed PAD47, PAD48: PAD-S-1.5, PADS:PAD-S-1.5
- added CON3: PINHEAD_1X02-2.54, pinhead:PINHEAD_1X02-2.54
- D1: value PTVS33VP1UTP,115-36V-SOD128 -> PTVS36VP1UP,115-36V-SOD128; device TVS_diodes:PTVS33VP1UTP,115-36V-SOD128 -> TVS_diodes:PTVS36VP1UP,115-36V-SOD128
- LED1: device rc:LED-0402 -> myxa_masterlib:LED-GREEN-0402
- LED2: device rc:LED-0402 -> myxa_masterlib:LED-GREEN-0402; COLOR GREEN -> (none); DIGIKEY# 1830-IN-S42BT5GCT-ND -> (none); MANF Inolux -> (none); MANF# IN-S42BT5G -> (none)
- LED3, LED4: device misc:LTST-C19HE1WT -> myxa_masterlib:LTST-C19HE1WT
- R10, R4: value 10 mOhms -> 5 mOhms; device SHUNT_RESISTORS:CURRENT_SHUNT_KELVIN-0.010R-2512-KELVIN -> SHUNT_RESISTORS:CURRENT_SHUNT_KELVIN-0.005R-2512-KELVIN
- R14: value 680R -> 1K; device rc:R-1%-0402 -> R_digikey:1K-1%-0402; AEC-Q AEC-Q200 -> (none); DIGIKEY# CRCW0402680RFKEDDatasheet -> (none); MANF Vishay Dale -> (none); MANF# CRCW0402680RFKED -> (none)
Connections:
- new net N$2: IC3.S
- net GND: now also CON3.1; no longer IC3.S, PAD47.P$1
- net GPIO1: now also CON3.2; no longer PAD48.P$1
Other:
- note added: "https://www.digikey.com/product-detail/en/united-chemi-con/EKZN500ELL181MH20D/565-4066-ND/4843876"
- note removed: "-Current shunts replaced (5 mOhms replaced with 10 mOhms)- -Overcurrent protection added. Itrip is ~35 A -RCPWM th connector replaced with smd solder pads -Some design notes added to the schematic -TVS diode (D1) replaced with one that has lower breaksdown voltage"
- note removed: "1.7"
- note removed: "100"
- note removed: "12"
- note removed: "14.4"
- note removed: "150"
- note removed: "200"
- note removed: "250"
- note removed: "3"
- note removed: "300"
- note removed: "4.5"
- note removed: "4.8"
- note removed: "6.3"
- note removed: "7.2"
- note removed: "8.4"
- note removed: "9.6"
- note removed: "97.2"
- note removed: "97.5"
- note removed: "97.7"
- note removed: "98"
- note removed: "98.3"
- note removed: "DC power, W"
- note removed: "Efficiency, %"
- note removed: "Phase current, I"
- note removed: "Power losses for different power levels"
- note removed: "R14 sets overcurrent protection trip level. 680R sets ir arount 35A, which is 2.5 times higher than maximum phase current for 300W DC power when running on discharged 8S battery"
- note removed: "The table is valid for 26.4 V supply voltage which is the same as a discharched 8S Li-ion battery"
- note removed: "Total losses, W"

Commit message: Bloxa V0.2
- Current shunts replaced (5 mOhms replaced with 10 mOhms)
- Overcurrent protection added. Itrip is ~35 A
- RCPWM th connector replaced with smd solder pads
- Some design notes added to the schematic
Parts:
- removed CON3: PINHEAD_1X02-2.54, pinhead:PINHEAD_1X02-2.54
- added PAD47, PAD48: PAD-S-1.5, PADS:PAD-S-1.5
- R10, R4: value 5 mOhms -> 10 mOhms; device SHUNT_RESISTORS:CURRENT_SHUNT_KELVIN-0.005R-2512-KELVIN -> SHUNT_RESISTORS:CURRENT_SHUNT_KELVIN-0.010R-2512-KELVIN
- R14: value 1K -> 680R; device R_digikey:1K-1%-0402 -> rc:R-1%-0402; AEC-Q (none) -> AEC-Q200; DIGIKEY# (none) -> CRCW0402680RFKEDDatasheet; MANF (none) -> Vishay Dale; MANF# (none) -> CRCW0402680RFKED
Connections:
- net GND: now also PAD47.P$1; no longer CON3.1
- net GPIO1: now also PAD48.P$1; no longer CON3.2
Other:
- note added: "1.7"
- note added: "100"
- note added: "12"
- note added: "14.4"
- note added: "150"
- note added: "200"
- note added: "250"
- note added: "3"
- note added: "300"
- note added: "4.5"
- note added: "4.8"
- note added: "6.3"
- note added: "7.2"
- note added: "8.4"
- note added: "9.6"
- note added: "97.2"
- note added: "97.5"
- note added: "97.7"
- note added: "98"
- note added: "98.3"
- note added: "DC power, W"
- note added: "Efficiency, %"
- note added: "Phase current, I"
- note added: "Power losses for different power levels"
- note added: "R14 sets overcurrent protection trip level. 680R sets ir arount 35A, which is 2.5 times higher than maximum phase current for 300W DC power when running on discharged 8S battery"
- note added: "The table is valid for 26.4 V supply voltage which is discharched 8S battery"
- note added: "Total losses, W"
- moved on the sheet: R14

Commit message: Some notes
Other:
- note added: "For 3d model check this link https://a360.co/3asTElW"
- note removed: "https://www.digikey.com/product-detail/en/united-chemi-con/EKZN500ELL181MH20D/565-4066-ND/4843876"

Commit message: changelog added as separate sheet to the schematic
Other:
- note added: "-Current shunts replaced (5 mOhms replaced with 10 mOhms)- -Overcurrent protection added. Itrip is ~35 A -RCPWM th connector replaced with smd solder pads -Some design notes added to the schematic"
Changed lines of the file:
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@@
 </attributes>
 <variantdefs>
-<variantdef name="Basic" current="yes"/>
+<variantdef name="Basic"/>
 <variantdef name="nocaps"/>
 </variantdefs>
@@
 <part name="PAD47" library="PADS" library_urn="urn:adsk.eagle:library:3188696" deviceset="PAD" device="-S-1.5" package3d_urn="urn:adsk.eagle:package:15477730/1"/>
 <part name="PAD48" library="PADS" library_urn="urn:adsk.eagle:library:3188696" deviceset="PAD" device="-S-1.5" package3d_urn="urn:adsk.eagle:package:15477730/1"/>
+<part name="FRAME2" library="frames" library_urn="urn:adsk.eagle:library:229" deviceset="A5L-LOC" device=""/>
 </parts>
 <sheets>
@@
 </nets>
 </sheet>
+<sheet>
+<description>changelog</description>
+<plain>
+<text x="7.62" y="101.6" size="1.778" layer="91" font="vector" align="center-left">-Current shunts replaced (5 mOhms replaced with 10 mOhms)-
+-Overcurrent protection added. Itrip is ~35 A
+-RCPWM th connector replaced with smd solder pads
+-Some design notes added to the schematic</text>
+</plain>
+<instances>
+<instance part="FRAME2" gate="G$1" x="0" y="0" smashed="yes">
+<attribute name="DRAWING_NAME" x="140.97" y="15.24" size="2.54" layer="94"/>
+<attribute name="LAST_DATE_TIME" x="140.97" y="10.16" size="2.286" layer="94"/>
+<attribute name="SHEET" x="154.305" y="5.08" size="2.54" layer="94"/>
+</instance>
+</instances>
+<busses>
+</busses>
+<nets>
+</nets>
+</sheet>

Commit message: ERC re-check
Connections:
- removed net N$2: IC3.S
- net GND: now also IC3.S
Other:
- note removed: "For 3d model check this link https://a360.co/3asTElW"
