File: bloxa.brd (EAGLE design)
At the start: 24.9 x 33.6 mm, 95 parts, among them CON1 CON-4P-JST_GH-RA, CON2 CON-4P-JST_GH-RA, IC1 MCP9700-SC70-5, IC2 TPD3S014DBVR-SOT23-6, IC3 TJA1051(X)/3-SO8, J1 CONNECTION, J2 CONNECTION, Q1 BUK9K6R2-40E,115, Q2 BUK9K6R2-40E,115, Q3 BUK9K6R2-40E,115

Commit message: attribute updated
Parts:
- D1: value PTVS36VP1UP,115-36V-SOD128 -> PTVS33VP1UTP,115-36V-SOD128
- LED1, LED2: device myxa_masterlib:0402_LED -> rc:LED0402
- LED3, LED4: device myxa_masterlib:LITE_ON_RGB_LED -> misc:0606
- turned LED1 to 0 degrees
- turned LED2 to 180 degrees
Routing:
- net GND: track 6.15 -> 8.20 mm, vias 10 -> 9

Commit message: resolving conflicts
Parts:
- removed PAD47, PAD48: PAD-S-1.5, PADS:1.5X1.5
- added CON3: PINHEAD_1X02-2.54, pinhead:1X02-PTH-2.54
- D1: value PTVS33VP1UTP,115-36V-SOD128 -> PTVS36VP1UP,115-36V-SOD128
- LED1, LED2: device rc:LED0402 -> myxa_masterlib:0402_LED
- LED3, LED4: device misc:0606 -> myxa_masterlib:LITE_ON_RGB_LED
- R10, R4: value 10 mOhms -> 5 mOhms
- R14: value 680R -> 1K; device rc:R0402 -> R_digikey:R0402
- turned LED1 to 180 degrees
- turned LED2 to 0 degrees
Connections:
- new net N$2: IC3.8
- net GND: now also CON3.1; no longer IC3.8, PAD47.P$1
- net GPIO1: now also CON3.2; no longer PAD48.P$1
Routing:
- net CAN1_VDD: track 29.4 -> 30.2 mm
- net GND: vias 9 -> 8
- removed copper zone on layer 1, net GND
Other:
- outline, holes or cut-outs redrawn
- board text added: "BLOXA 0.1"
- board text added: "Replace CON3 with SMD pads. No TH components allowed here"
- board text removed: "BLOXA 0.2"

Commit message: Hardware files updated
Parts:
- removed CON3: PINHEAD_1X02-2.54, pinhead:1X02-PTH-2.54
- added PAD47, PAD48: PAD-S-1.5, PADS:1.5X1.5
- D1: value PTVS36VP1UP,115-36V-SOD128 -> PTVS33VP1UTP,115-36V-SOD128
- LED1, LED2: device myxa_masterlib:0402_LED -> rc:LED0402
- LED3, LED4: device myxa_masterlib:LITE_ON_RGB_LED -> misc:0606
- R10, R4: value 5 mOhms -> 10 mOhms
- R14: value 1K -> 680R; device R_digikey:R0402 -> rc:R0402
- turned LED1 to 0 degrees
- turned LED2 to 180 degrees
Connections:
- removed net N$2: IC3.8
- net GND: now also IC3.8, PAD47.P$1; no longer CON3.1
- net GPIO1: now also PAD48.P$1; no longer CON3.2
Routing:
- net CAN1_VDD: track 30.2 -> 29.4 mm
- net GND: vias 8 -> 9
- added copper zone on layer 1, net GND
Other:
- outline, holes or cut-outs redrawn
- board text added: "BLOXA 0.2"
- board text removed: "BLOXA 0.1"
- board text removed: "Replace CON3 with SMD pads. No TH components allowed here"
